Commit message: modifica per la posizione del file

File: uav_navigation/src/drone_planning/model/iris2/iris1.urdf (robot description, URDF)
Before this commit: robot iris, 6 links, 5 joints
Links:
- link base_link: geometry collision box size=0.47 0.47 0.11; visual mesh filename=file:///home/test/uav_navigation/src/drone_planning/model/i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 scale=1 1 1
- link iris__rotor_0: geometry collision cylinder length=0.005 radius=0.128; visual mesh filename=file:///home/test/uav_navigation/src/drone_planning/model/i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 scale=1 1 1
- link iris__rotor_1: geometry collision cylinder length=0.005 radius=0.128; visual mesh filename=file:///home/test/uav_navigation/src/drone_planning/model/i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 scale=1 1 1
- link iris__rotor_2: geometry collision cylinder length=0.005 radius=0.128; visual mesh filename=file:///home/test/uav_navigation/src/drone_planning/model/i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 scale=1 1 1
- link iris__rotor_3: geometry collision cylinder length=0.005 radius=0.128; visual mesh filename=file:///home/test/uav_navigation/src/drone_planning/model/i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 scale=1 1 1

Commit message: modifica file urdf per pc qualsiasi

File: uav_navigation/src/drone_planning/model/iris2/iris1.urdf (robot description, URDF)
Before this commit: robot iris, 6 links, 5 joints
Links:
- link base_link: geometry collision box size=0.47 0.47 0.11; visual mesh filename=package://drone_planning/model/iris2/iris1.dae scale=1 1 1
- link iris__rotor_0: geometry collision cylinder length=0.005 radius=0.128; visual mesh filename=package://drone_planning/model/iris2/iris_prop_ccw.dae scale=1 1 1
- link iris__rotor_1: geometry collision cylinder length=0.005 radius=0.128; visual mesh filename=package://drone_planning/model/iris2/iris_prop_ccw.dae scale=1 1 1
- link iris__rotor_2: geometry collision cylinder length=0.005 radius=0.128; visual mesh filename=package://drone_planning/model/iris2/iris_prop_cw.dae scale=1 1 1
- link iris__rotor_3: geometry collision cylinder length=0.005 radius=0.128; visual mesh filename=package://drone_planning/model/iris2/iris_prop_cw.dae scale=1 1 1
